File: hardware/out/hub/slimevr-i2spi-hub.kicad_sch (KiCad schematic)
At the start: 33 parts, among them J1 RJ45-CHAIN, J2 LiPo, J3 USB-C, SW1 BOOT, U1 ESP32-C5-WROOM-1, U2 ICM-45686, U3 QMC6309, U4 AP2112K-3.3, U5 MCP73831

Commit message: Vendor Espressif and Mumo KiCad libraries; document I2SPI
docs/I2SPI.md consolidates the RJ45 pinout and the v2 wire protocol.

Espressif's own C5 symbol corrected a live bug: BOARD_SLIMEVR_C5_CHAIN_HUB had SPI
MISO/MOSI on GPIO11/GPIO12, which are U0TXD/U0RXD on the module. Moved to GPIO9/8,
INT to 15, LED to 23.

QMC6309 is a 4-pad WLCSP, not the DFN-6 the placeholder assumed. Both parts now
sourced from vendored libraries. ICM-45686 remains the only unverified pinout.
Parts:
- removed U1: ESP32-C5-WROOM-1, slimevr-i2spi:ESP32-C5-WROOM-1, symbol slimevr-i2spi:ESP32-C5-WROOM-1
- removed U3: QMC6309, slimevr-i2spi:DFN-6_1.6x1.6mm_P0.5mm, symbol slimevr-i2spi:QMC6309
- added U1: ESP32-C5-WROOM-1, Espressif:ESP32-C5-WROOM-1, symbol Espressif:ESP32-C5-WROOM-1
- added U3: QMC6309, Mumo:QMC6309, symbol Mumo:QMC6309
Changed lines of the file:
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@@
     (comment 2 "ESP32-C5, local IMU, battery, one chain port")
   )
-  (symbol (lib_id "slimevr-i2spi:ESP32-C5-WROOM-1") (at 38.10 38.10 0) (unit 1)
+  (symbol (lib_id "Espressif:ESP32-C5-WROOM-1") (at 38.10 38.10 0) (unit 1)
     (in_bom yes) (on_board yes)
     (property "Reference" "U1" (at 38.10 25.40 0)
@@
     (property "Value" "ESP32-C5-WROOM-1" (at 38.10 50.80 0)
       (effects (font (size 1.27 1.27))))
-    (property "Footprint" "slimevr-i2spi:ESP32-C5-WROOM-1" (at 38.10 38.10 0)
+    (property "Footprint" "Espressif:ESP32-C5-WROOM-1" (at 38.10 38.10 0)
       (effects (font (size 1.27 1.27)) hide))
     (property "LCSC" "C5736265" (at 38.10 38.10 0)
@@
     (effects (font (size 1.27 1.27)) (justify left))
   )
-  (symbol (lib_id "slimevr-i2spi:QMC6309") (at 165.10 38.10 0) (unit 1)
+  (symbol (lib_id "Mumo:QMC6309") (at 165.10 38.10 0) (unit 1)
     (in_bom yes) (on_board yes)
     (property "Reference" "U3" (at 165.10 25.40 0)
@@
     (property "Value" "QMC6309" (at 165.10 50.80 0)
       (effects (font (size 1.27 1.27))))
-    (property "Footprint" "slimevr-i2spi:DFN-6_1.6x1.6mm_P0.5mm" (at 165.10 38.10 0)
+    (property "Footprint" "Mumo:QMC6309" (at 165.10 38.10 0)
       (effects (font (size 1.27 1.27)) hide))
     (property "LCSC" "C5325803" (at 165.10 38.10 0)

Commit message: Verification audit: fix CCL LUT number, strip fabricated part numbers
Checked ~30 load-bearing claims against primary sources. Four were wrong, two
were live:

- PA7 on an 8-pin tinyAVR is LUT1-OUT, not LUT0's alternate (LUT0-OUT is PA4,
  absent from the package). The node firmware configured Logic0, whose output
  cannot reach a pin, so the strobe pass-through would not have worked.
- Every LCSC part number was fabricated. The one checkable is wrong. Stripped to
  None so the BOM fails at upload rather than at assembly.
- ICM-45686 draws 0.42 mA in 6-axis low-noise mode, not the 2.5 mA estimated.

Verified correct: all ESP32-C5 GPIO restrictions, boot-mode pins, ADC placement,
the IMU package and AUX port, TWI pin fixing on 8-pin parts, and the QEMU and
ATtiny10 exclusions.
Parts:
- D1, D2: LCSC C2286 -> (none)
- J1: LCSC C86550 -> (none)
- J3: LCSC C165948 -> (none)
- U1: LCSC C5736265 -> (none)
- U2: LCSC C5457057 -> (none)
- U3: LCSC C5325803 -> (none)
- U4: LCSC C51118 -> (none)
- U5: LCSC C424093 -> (none)
Changed lines of the file:
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@@
     (property "Footprint" "Espressif:ESP32-C5-WROOM-1" (at 38.10 38.10 0)
       (effects (font (size 1.27 1.27)) hide))
-    (property "LCSC" "C5736265" (at 38.10 38.10 0)
-      (effects (font (size 1.27 1.27)) hide))
     (property "Note" "dual-band; band selected explicitly at runtime, see DEC-002" (at 38.10 38.10 0)
       (effects (font (size 1.27 1.27)) hide))
@@
     (property "Footprint" "slimevr-i2spi:LGA-14_2.5x3mm_P0.5mm" (at 101.60 38.10 0)
       (effects (font (size 1.27 1.27)) hide))
-    (property "LCSC" "C5457057" (at 101.60 38.10 0)
-      (effects (font (size 1.27 1.27)) hide))
     (property "Note" "hub's own IMU - NOT power gated, and its CS never leaves the board" (at 101.60 38.10 0)
       (effects (font (size 1.27 1.27)) hide))
@@
     (property "Footprint" "Mumo:QMC6309" (at 165.10 38.10 0)
       (effects (font (size 1.27 1.27)) hide))
-    (property "LCSC" "C5325803" (at 165.10 38.10 0)
-      (effects (font (size 1.27 1.27)) hide))
   )
   (global_label "AUX_SCL" (shape bidirectional) (at 182.88 27.94 0)
@@
     (property "Footprint" "Connector_RJ:RJ45_Amphenol_54602-x08_Horizontal" (at 228.60 38.10 0)
       (effects (font (size 1.27 1.27)) hide))
-    (property "LCSC" "C86550" (at 228.60 38.10 0)
-      (effects (font (size 1.27 1.27)) hide))
     (property "Note" "to the sensor chain" (at 228.60 38.10 0)
       (effects (font (size 1.27 1.27)) hide))
@@
     (property "Footprint" "Package_TO_SOT_SMD:SOT-23-5" (at 228.60 114.30 0)
       (effects (font (size 1.27 1.27)) hide))
-    (property "LCSC" "C51118" (at 228.60 114.30 0)
-      (effects (font (size 1.27 1.27)) hide))
   )
   (global_label "VBAT" (shape bidirectional) (at 246.38 104.14 0)
@@
     (property "Footprint" "Package_TO_SOT_SMD:SOT-23-5" (at 38.10 152.40 0)
       (effects (font (size 1.27 1.27)) hide))
-    (property "LCSC" "C424093" (at 38.10 152.40 0)
-      (effects (font (size 1.27 1.27)) hide))
   )
   (global_label "VUSB" (shape bidirectional) (at 55.88 142.24 0)
@@
     (property "Footprint" "LED_SMD:LED_0603_1608Metric" (at 101.60 190.50 0)
       (effects (font (size 1.27 1.27)) hide))
-    (property "LCSC" "C2286" (at 101.60 190.50 0)
-      (effects (font (size 1.27 1.27)) hide))
   )
   (global_label "LED" (shape bidirectional) (at 119.38 180.34 0)
@@
     (property "Footprint" "Connector_USB:USB_C_Receptacle_HRO_TYPE-C-31-M-12" (at 38.10 304.80 0)
       (effects (font (size 1.27 1.27)) hide))
-    (property "LCSC" "C165948" (at 38.10 304.80 0)
-      (effects (font (size 1.27 1.27)) hide))
     (property "Note" "charge and flash" (at 38.10 304.80 0)
       (effects (font (size 1.27 1.27)) hide))
@@
     (property "Footprint" "LED_SMD:LED_0603_1608Metric" (at 228.60 304.80 0)
       (effects (font (size 1.27 1.27)) hide))
-    (property "LCSC" "C2286" (at 228.60 304.80 0)
-      (effects (font (size 1.27 1.27)) hide))
     (property "Note" "charge status" (at 228.60 304.80 0)
