File: hardware/out/node/slimevr-i2spi-node.kicad_sch (KiCad schematic)
At the start: 16 parts, among them J1 RJ45-IN, J2 RJ45-OUT, Q1 DMG2305UX, U1 ATtiny412, U2 ICM-45686, U3 QMC6309

Commit message: Vendor Espressif and Mumo KiCad libraries; document I2SPI
docs/I2SPI.md consolidates the RJ45 pinout and the v2 wire protocol.

Espressif's own C5 symbol corrected a live bug: BOARD_SLIMEVR_C5_CHAIN_HUB had SPI
MISO/MOSI on GPIO11/GPIO12, which are U0TXD/U0RXD on the module. Moved to GPIO9/8,
INT to 15, LED to 23.

QMC6309 is a 4-pad WLCSP, not the DFN-6 the placeholder assumed. Both parts now
sourced from vendored libraries. ICM-45686 remains the only unverified pinout.
Parts:
- removed U3: QMC6309, slimevr-i2spi:DFN-6_1.6x1.6mm_P0.5mm, symbol slimevr-i2spi:QMC6309
- added U3: QMC6309, Mumo:QMC6309, symbol Mumo:QMC6309
Changed lines of the file:
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@@
     (effects (font (size 1.27 1.27)) (justify left))
   )
-  (symbol (lib_id "slimevr-i2spi:QMC6309") (at 165.10 76.20 0) (unit 1)
+  (symbol (lib_id "Mumo:QMC6309") (at 165.10 76.20 0) (unit 1)
     (in_bom yes) (on_board yes)
     (property "Reference" "U3" (at 165.10 63.50 0)
@@
     (property "Value" "QMC6309" (at 165.10 88.90 0)
       (effects (font (size 1.27 1.27))))
-    (property "Footprint" "slimevr-i2spi:DFN-6_1.6x1.6mm_P0.5mm" (at 165.10 76.20 0)
+    (property "Footprint" "Mumo:QMC6309" (at 165.10 76.20 0)
       (effects (font (size 1.27 1.27)) hide))
     (property "LCSC" "C5325803" (at 165.10 76.20 0)

Commit message: Verification audit: fix CCL LUT number, strip fabricated part numbers
Checked ~30 load-bearing claims against primary sources. Four were wrong, two
were live:

- PA7 on an 8-pin tinyAVR is LUT1-OUT, not LUT0's alternate (LUT0-OUT is PA4,
  absent from the package). The node firmware configured Logic0, whose output
  cannot reach a pin, so the strobe pass-through would not have worked.
- Every LCSC part number was fabricated. The one checkable is wrong. Stripped to
  None so the BOM fails at upload rather than at assembly.
- ICM-45686 draws 0.42 mA in 6-axis low-noise mode, not the 2.5 mA estimated.

Verified correct: all ESP32-C5 GPIO restrictions, boot-mode pins, ADC placement,
the IMU package and AUX port, TWI pin fixing on 8-pin parts, and the QEMU and
ATtiny10 exclusions.
Parts:
- J1, J2: LCSC C86550 -> (none)
- Q1: LCSC C111885 -> (none)
- U1: LCSC C79945 -> (none)
- U2: LCSC C5457057 -> (none)
- U3: LCSC C5325803 -> (none)
Changed lines of the file:
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@@
     (property "Footprint" "Connector_RJ:RJ45_Amphenol_54602-x08_Horizontal" (at 38.10 38.10 0)
-      (effects (font (size 1.27 1.27)) hide))
-    (property "LCSC" "C86550" (at 38.10 38.10 0)
       (effects (font (size 1.27 1.27)) hide))
     (property "Note" "chain in" (at 38.10 38.10 0)
@@
     (property "Footprint" "Connector_RJ:RJ45_Amphenol_54602-x08_Horizontal" (at 101.60 38.10 0)
       (effects (font (size 1.27 1.27)) hide))
-    (property "LCSC" "C86550" (at 101.60 38.10 0)
-      (effects (font (size 1.27 1.27)) hide))
     (property "Note" "chain out - wired pin-for-pin in parallel with J1, zero-length stub" (at 101.60 38.10 0)
       (effects (font (size 1.27 1.27)) hide))
@@
     (property "Footprint" "Package_SO:SOIC-8_3.9x4.9mm_P1.27mm" (at 165.10 38.10 0)
       (effects (font (size 1.27 1.27)) hide))
-    (property "LCSC" "C79945" (at 165.10 38.10 0)
-      (effects (font (size 1.27 1.27)) hide))
     (property "Note" "I2SPI controller" (at 165.10 38.10 0)
       (effects (font (size 1.27 1.27)) hide))
@@
       (effects (font (size 1.27 1.27))))
     (property "Footprint" "Package_TO_SOT_SMD:SOT-23" (at 228.60 38.10 0)
-      (effects (font (size 1.27 1.27)) hide))
-    (property "LCSC" "C111885" (at 228.60 38.10 0)
       (effects (font (size 1.27 1.27)) hide))
     (property "Note" "high-side pass FET: gate low = sensor powered" (at 228.60 38.10 0)
@@
       (effects (font (size 1.27 1.27))))
     (property "Footprint" "slimevr-i2spi:LGA-14_2.5x3mm_P0.5mm" (at 101.60 76.20 0)
-      (effects (font (size 1.27 1.27)) hide))
-    (property "LCSC" "C5457057" (at 101.60 76.20 0)
       (effects (font (size 1.27 1.27)) hide))
     (property "Note" "gated supply; INT pins deliberately unconnected, see DEC-004" (at 101.60 76.20 0)
@@
     (property "Footprint" "Mumo:QMC6309" (at 165.10 76.20 0)
       (effects (font (size 1.27 1.27)) hide))
-    (property "LCSC" "C5325803" (at 165.10 76.20 0)
-      (effects (font (size 1.27 1.27)) hide))
     (property "Note" "on the IMU AUX1 bus, not the chain" (at 165.10 76.20 0)
